File: projects/STM32F4-PCB/pcb/STM32F4_REV2.kicad_pcb (KiCad board)
At the start: 4 copper layers, 56 x 51 mm, 54 parts, among them J1 Screw_Terminal_01x02, J2 SWD, J3 Conn_01x04, J4 Conn_01x04, J5 USB_B_Micro, Q1 AO3401A, SW1 SW_SPDT, U1 MP2359DJ-LF-Z, U2 STM32F405RGT6, U3 USBLC6-2SC6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

Commit message: repo updated
Other:
- net class Default removed
