File: stm32_prototype/stm32_prototype.kicad_pcb (KiCad board)
At the start: 2 copper layers, 70 x 50 mm, 103 parts, among them J1 XT30 battery 2S-3S, J10 RC3, J11 LIGHT1, J12 LIGHT2, J13 Cortex-Debug, J14 Qwiic, J15 UART, J16 EXPANSION, J2 USB-C, J3 MOTOR, J4 SERVO1, J5 SERVO2, J6 SERVO3, J7 SERVO4, J8 RC1, J9 RC2, Q1 AO4407A, Q2 AO3400A, Q3 AO3400A, SW1 BOOT0, SW2 RESET, U1 STM32F103C8T6, U2 TPS563201, U3 USBLC6-2SC6, U4 AP2112K-3.3, U5 DRV8870, U6 LSM6DS3TR-C, Y1 8MHz, Y2 32.768kHz

Commit message: Rev C routing: 4 layers SIG/GND/SIG/SIG, solid In1 GND plane, bottom silk labels
- Freerouting on F.Cu/In2/B.Cu with GND as an In1 plane; In1 made 30x more expensive
  in a rules file so it only receives vias and stays one solid plane
- GND pours on all layers, edge stitching; battery/motor/servo nets 0.8 mm
- Bottom silkscreen: servo/receiver/light/UART pin functions, battery polarity
- DRC: 0 violations, 0 unconnected, 0 schematic parity issues

Co-Authored-By: Claude Opus 5.5 (1M context) <noreply@anthropic.com>
Parts:
- moved J16 47.4 mm to (148.5, 102.0)
- moved C27 21.3 mm to (133.6, 145.6)
- moved J3 20.0 mm to (111.0, 144.0)
- turned U5 to 180 degrees
Routing:
- net GND: track 0.00 -> 234.4 mm, vias 0 -> 85
- net +3V3: track 0.00 -> 217.6 mm, vias 0 -> 7
- net V5_SERVO: track 0.00 -> 87.0 mm, vias 0 -> 1
- net VBAT: track 0.00 -> 86.5 mm, vias 0 -> 6
- net NRST: track 0.00 -> 60.7 mm, vias 0 -> 4
- net SERVO1: track 0.00 -> 58.8 mm, vias 0 -> 1
- net SERVO3: track 0.00 -> 52.6 mm, vias 0 -> 1
- net I2C_SDA: track 0.00 -> 51.1 mm, vias 0 -> 3
- net SERVO2: track 0.00 -> 50.8 mm, vias 0 -> 1
- net +5V: track 0.00 -> 48.5 mm, vias 0 -> 3
- net PA5: track 0.00 -> 47.3 mm, vias 0 -> 1
- net I2C_SCL: track 0.00 -> 47.2 mm, vias 0 -> 4
- net /MCU/BOOT0: track 0.00 -> 45.0 mm, vias 0 -> 3
- net VBAT_SENSE: track 0.00 -> 44.7 mm, vias 0 -> 2
- net SERVO4: track 0.00 -> 41.7 mm, vias 0 -> 1
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- added copper zone on B.Cu, net GND
- added copper zone on F.Cu, net GND
- added copper zone on In1.Cu, net GND
- added copper zone on In2.Cu, net GND
Other:
- copper layers 2 -> 4
- board text added: "+"
- board text added: "+ BATT -"
- board text added: "-"
- board text added: "2S-3S LiPo"
- board text added: "5V"
- board text added: "BOOT0"
- board text added: "EXPANSION"
- board text added: "GND"
- board text added: "L1"
- board text added: "L2"
- board text added: "MOTOR"
- board text added: "QWIIC"
- board text added: "R1"
- board text added: "R2"
- board text added: "R3"
- board text added: "RESET"
- board text added: "RX"
- board text added: "S"
- board text added: "S1"
- board text added: "S2"
- board text added: "S3"
- board text added: "S4"
- board text added: "STM32 RC controller Rev C"
- board text added: "SWD"
- board text added: "TX"
- board text added: "USB-C"
