File: stm32_prototype/stm32_prototype.kicad_pcb (KiCad board)
At the start: 4 copper layers, 70 x 50 mm, 103 parts, among them J1 XT30 battery 2S-3S, J10 RC3, J11 LIGHT1, J12 LIGHT2, J13 Cortex-Debug, J14 Qwiic, J15 UART, J16 EXPANSION, J2 USB-C, J3 MOTOR, J4 SERVO1, J5 SERVO2, J6 SERVO3, J7 SERVO4, J8 RC1, J9 RC2, Q1 AO4407A, Q2 AO3400A, Q3 AO3400A, SW1 BOOT0, SW2 RESET, U1 STM32F103C8T6, U2 TPS563201, U3 USBLC6-2SC6, U4 AP2112K-3.3, U5 DRV8870, U6 LSM6DS3TR-C, Y1 8MHz, Y2 32.768kHz

Commit message: Rev C: WS2812 RGB lighting output for 6 LEDs
- PA8 (TIM1 CH1 + DMA) -> SN74AHCT1G125 at 5 V -> 330R -> 3-pin connector (5V, DIN, GND),
  22 uF at the connector; PA8 removed from the expansion header
- Board re-placed and re-routed: DRC 0 violations, 0 unconnected, 0 parity issues; bottom silk 'RGB 5V DI G'
- Firmware: 800 kHz WS2812 driver via DMA, default head/sill/tail colours, 'c' colour and 'ind' indicator
  commands; builds (30 KB flash)
- Fabrication data, schematic images, renders and docs updated

Co-Authored-By: Claude Opus 5.5 (1M context) <noreply@anthropic.com>
Parts:
- added C33: 100n, Capacitor_SMD:C_0603_1608Metric, F.Cu at (103.5, 120.5)
- added C34: 22u 25V, Capacitor_SMD:C_1206_3216Metric, F.Cu at (107.0, 111.0)
- added J17: WS2812, Connector_PinHeader_2.54mm:PinHeader_1x03_P2.54mm_Vertical, F.Cu at (103.0, 109.5)
- added R29: 330R, Resistor_SMD:R_0603_1608Metric, F.Cu at (107.5, 121.5)
- added U7: SN74AHCT1G125, Package_TO_SOT_SMD:SOT-23-5, F.Cu at (107.5, 117.5)
Connections:
- J16 pad 4: PA8 -> GND
- U1 pad 29: PA8 -> LED_DATA
Routing:
- net LED_DATA: track 0.00 -> 50.2 mm, vias 0 -> 2
- net +5V: track 48.5 -> 91.6 mm, vias 3 -> 4
- net PA8: track 30.3 -> 0.00 mm, vias 2 -> 0
- net GND: track 234.4 -> 263.2 mm, vias 85 -> 81
- net +3V3: track 217.6 -> 198.6 mm
- net LIGHT2: track 24.2 -> 41.2 mm
- net /IO/LED_DIN: track 0.00 -> 15.8 mm
- net PA5: track 47.3 -> 32.4 mm
- net SWDIO: track 31.7 -> 21.0 mm
- net SERVO1: track 58.8 -> 69.4 mm
- net /MCU/BOOT0: track 45.0 -> 54.8 mm, vias 3 -> 2
- net VBUS: track 28.6 -> 19.6 mm, vias 2 -> 4
- net PB9: track 28.7 -> 36.8 mm, vias 2 -> 1
- net V5_SERVO: track 87.0 -> 94.6 mm, vias 1 -> 2
- net I2C_SCL: track 47.2 -> 54.3 mm, vias 4 -> 5
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Other:
- board text added: "DI"
- board text added: "G"
- board text added: "RGB"
